File: pow3.5e2.brd (EAGLE design)
At the start: 99.7 x 69.8 mm, 66 parts, among them X1 FH12-20S-1SH, X2 JST-2-PXH, X3 JST-2-PXH

Commit message: Update pow3.5e2.brd
Routing:
- net GND: track 37.1 -> 39.7 mm
- net RT: track 18.2 -> 19.7 mm

Commit message: sch
Routing:
- net GND: track 39.7 -> 41.2 mm
Changed lines of the file:
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@@
 <layer number="28" name="bValues" color="7" fill="1" visible="no" active="yes"/>
 <layer number="29" name="tStop" color="7" fill="3" visible="no" active="yes"/>
-<layer number="30" name="bStop" color="7" fill="6" visible="no" active="yes"/>
+<layer number="30" name="bStop" color="7" fill="6" visible="yes" active="yes"/>
 <layer number="31" name="tCream" color="7" fill="4" visible="no" active="yes"/>
 <layer number="32" name="bCream" color="7" fill="5" visible="no" active="yes"/>
@@
 <layer number="220" name="220bmp" color="7" fill="1" visible="no" active="yes"/>
 <layer number="221" name="221bmp" color="7" fill="1" visible="no" active="yes"/>
+<layer number="222" name="222bmp" color="7" fill="1" visible="no" active="yes"/>
 <layer number="223" name="223bmp" color="7" fill="1" visible="no" active="yes"/>
 <layer number="224" name="224bmp" color="7" fill="1" visible="no" active="yes"/>
@@
 <vertex x="8.89" y="8.5725"/>
 <vertex x="12.065" y="11.7475"/>
-<vertex x="12.065" y="33.9725"/>
-<vertex x="-8.255" y="33.9725"/>
+<vertex x="12.065" y="34.29"/>
+<vertex x="-8.255" y="34.29"/>
 <vertex x="-8.255" y="36.195"/>
 </polygon>
@@
 <contactref element="X1" pad="8"/>
 <wire x1="-1.055" y1="24.3725" x2="-1.055" y2="25.669475" width="0.4064" layer="16"/>
-<wire x1="-1.055" y1="25.669475" x2="-0.8690125" y2="26.1184875" width="0.4064" layer="16" curve="-45"/>
 <wire x1="-2.2225" y1="17.181" x2="-2.2225" y2="15.71625" width="0.4064" layer="16"/>
 <via x="7.62" y="20.6375" extent="1-16" drill="0.508"/>
@@
 <wire x1="-1.215525" y1="27.041975" x2="-1.5875" y2="26.14395" width="0.4064" layer="16" curve="45"/>
 <wire x1="-1.5875" y1="26.14395" x2="-1.5875" y2="26.035" width="0.4064" layer="16"/>
+<wire x1="-2.0075" y1="25.669475" x2="-1.8215125" y2="25.9597375" width="0.4064" layer="16" curve="-45"/>
+<wire x1="-1.476775" y1="25.97875" x2="-1.1865125" y2="25.7927625" width="0.4064" layer="16" curve="-45"/>
+<wire x1="1.96125" y1="23.26125" x2="1.96125" y2="24.38875" width="0.4064" layer="16"/>
+<wire x1="1.96125" y1="24.4475" x2="1.96125" y2="24.558225" width="0.4064" layer="16"/>
+<wire x1="1.945" y1="24.3725" x2="1.96125" y2="24.38875" width="0.4064" layer="16" curve="90"/>
+<wire x1="1.96125" y1="24.38875" x2="1.96125" y2="24.4475" width="0.4064" layer="16"/>
 </signal>
 <signal name="/FAN">
