File: pow3.5e2.sch (EAGLE design)
At the start: 66 parts, among them X1 FH12-20S-1SH, X2 JST-2-PXH, X3 JST-2-PXH

Commit message: sch
Other:
- note added: "MKlon3.5 pow3.5eX"
- note added: "Olmoro 2024"
- note removed: "mklon3.5 pow3.5vX"
Changed lines of the file:
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@@
 <sheet>
 <plain>
-<text x="175.26" y="7.62" size="3.81" layer="94">mklon3.5
-pow3.5vX</text>
+<text x="175.26" y="7.62" size="3.81" layer="94">MKlon3.5
+pow3.5eX</text>
 <wire x1="63.5" y1="34.29" x2="58.42" y2="34.29" width="0.1524" layer="94"/>
 <wire x1="58.42" y1="34.29" x2="58.42" y2="35.56" width="0.1524" layer="94"/>
@@
 <text x="15.24" y="157.48" size="2.54" layer="91" font="vector" ratio="10" align="center">+19V</text>
 <text x="15.24" y="142.24" size="2.54" layer="91" font="vector" ratio="10" align="center">-19V</text>
+<text x="236.22" y="20.32" size="2.54" layer="94" font="vector" ratio="14" align="bottom-center">Olmoro 2024</text>
 </plain>
 <instances>
